File: PRetvornik_ohisja/LFCSP_2_DIP.sch (KiCad schematic (older format))
At the start: 3 parts, among them P1 CONN_01X08, P2 CONN_01X08, U1 ADCMP572

Commit message: Naredil nov LFCSP s osrednjim padom in ga zavrtel za 45 stopinj
Parts:
- P1, P2: footprint w_pin_strip:pin_socket_8 -> Socket_Strips:Socket_Strip_Straight_1x08_Pitch2.54mm
- U1: footprint mitja:QFP_16 -> LFCSP:LFCSP_45
Changed lines of the file:
@@
 LIBS:valves
 LIBS:adcmp572
+LIBS:LFCSP_2_DIP-cache
 EELAYER 25 0
 EELAYER END
@@
 F 0 "U1" H 3400 2900 60  0000 C CNN
 F 1 "ADCMP572" H 3750 2550 60  0000 C CNN
-F 2 "mitja:QFP_16" H 3750 2550 60  0001 C CNN
+F 2 "LFCSP:LFCSP_45" H 3750 2550 60  0001 C CNN
 F 3 "" H 3750 2550 60  0000 C CNN
 	1    3350 2850
@@
 F 0 "P1" H 4900 3500 50  0000 C CNN
 F 1 "CONN_01X08" V 5000 3050 50  0000 C CNN
-F 2 "w_pin_strip:pin_socket_8" H 4900 3050 50  0001 C CNN
+F 2 "Socket_Strips:Socket_Strip_Straight_1x08_Pitch2.54mm" H 4900 3050 50  0001 C CNN
 F 3 "" H 4900 3050 50  0000 C CNN
 	1    4900 3050
@@
 F 0 "P2" H 5500 3500 50  0000 C CNN
 F 1 "CONN_01X08" V 5600 3050 50  0000 C CNN
-F 2 "w_pin_strip:pin_socket_8" H 5500 3050 50  0001 C CNN
+F 2 "Socket_Strips:Socket_Strip_Straight_1x08_Pitch2.54mm" H 5500 3050 50  0001 C CNN
 F 3 "" H 5500 3050 50  0000 C CNN
 	1    5500 3050
